Commit message: Controlleur tuto fonctionnel

File: pa_ctrl/workcell_moveit_config/config/gazebo_fanuc_crx10ial.urdf (robot description, URDF)
Before this commit: robot fanuc_crx10ial, 16 links, 15 joints
Joints:
- joint joint_1: limit lower=-3.141592653589793 upper=3.141592653589793 effort=0 velocity=2.0943951023931953 -> lower=-3.141592653589793 upper=3.141592653589793 effort=100 velocity=2.0943951023931953
- joint joint_3: limit lower=-4.71238898038469 upper=4.71238898038469 effort=0 velocity=3.141592653589793 -> lower=-4.71238898038469 upper=4.71238898038469 effort=100 velocity=3.141592653589793
- joint joint_4: limit lower=-3.3161255787892263 upper=3.3161255787892263 effort=0 velocity=3.141592653589793 -> lower=-3.3161255787892263 upper=3.3161255787892263 effort=100 velocity=3.141592653589793
- joint joint_5: limit lower=-3.141592653589793 upper=3.141592653589793 effort=0 velocity=3.141592653589793 -> lower=-3.141592653589793 upper=3.141592653589793 effort=100 velocity=3.141592653589793
- joint joint_6: limit lower=-3.3161255787892263 upper=3.3161255787892263 effort=0 velocity=3.141592653589793 -> lower=-3.3161255787892263 upper=3.3161255787892263 effort=100 velocity=3.141592653589793
