Commit message: ajout move avec cpp

File: pa_ctrl/pa_ctrl/urdf/workcell.urdf (robot description, URDF)
Before this commit: robot fanuc_crx10ial, 13 links, 12 joints
Links:
- added link TCP; visual sphere radius=0.005
- added link camera_frame
- added link world
- link robot_base_plate: geometry collision box size=0.35 0.2 0.01; visual mesh filename=package://pa_ctrl/rviz/meshes/visual/base_plate.dae
Joints:
- added joint festool_kit_to_TCP: type fixed, parent festool_kit, child TCP, origin xyz=0 -0.020860 0.141701 rpy=0 0 0
- added joint world_to_camera: type fixed, parent world, child camera_frame, origin xyz=-0.25 -0.5 1.25 rpy=0 3.14159 0
- added joint world_to_husky: type fixed, parent world, child husky, origin xyz=0 0 0 rpy=0 0 0
- joint husky_to_robot_base_plate: origin (none) -> xyz=0.0 0.0 0.798396 rpy=0 0 0
- joint robot_base_plate_to_base_link: origin (none) -> xyz=0 0 0 rpy=0 0 0
- joint tool0_to_festool_kit: origin (none) -> xyz=0 0 0 rpy=0 0 0

File: pa_ctrl/pa_ctrl/urdf/workcell.xacro (robot description, xacro)
@@ -55,4 +55,6 @@
     </visual>
   </link>
+  <link name="world"/>
+  <link name="camera_frame"/>
   <!-- Diefine joint between link-->
   <joint name="tool0_to_festool_kit" type="fixed">
@@ -79,8 +81,13 @@
     <child  link="TCP"/>
   </joint>
-  <!--joint name="world_to_husky" type="fixed">
+  <joint name="world_to_husky" type="fixed">
     <origin xyz="0 0 0" rpy="0 0 0" />
     <parent link="world"/>
     <child  link="husky"/>
-  </joint-->
+  </joint>
+  <joint name="world_to_camera" type="fixed">
+    <parent link="world"/>
+    <child link="camera_frame"/>
+    <origin xyz="-0.25 -0.5 1.25" rpy="0 3.14159 0"/>
+  </joint>
 </robot>

File: pa_ctrl/workcell_moveit_config/config/gazebo_fanuc_crx10ial.urdf (robot description, URDF)
Before this commit: robot fanuc_crx10ial, 14 links, 13 joints
Links:
- added link camera_frame
- added link world
Joints:
- added joint world_to_camera: type fixed, parent world, child camera_frame, origin xyz=-0.25 -0.5 1.25 rpy=0 3.14159 0
- added joint world_to_husky: type fixed, parent world, child husky, origin xyz=0 0 0 rpy=0 0 0

Commit message: descarte planner avec fake ar -- IKFast intermittant

File: pa_ctrl/pa_ctrl/urdf/workcell.urdf (robot description, URDF)
Before this commit: robot fanuc_crx10ial, 16 links, 15 joints
Links:
- link festool_kit: geometry collision mesh filename=package://pa_ctrl/rviz/meshes/collision/Festool_colision.stl; visual mesh filename=package://pa_ctrl/rviz/meshes/visual/Festool_v4.stl
- link husky: geometry collision mesh filename=package://pa_ctrl/rviz/meshes/collision/collision_mesh.stl; visual mesh filename=package://pa_ctrl/rviz/meshes/visual/base_mobile.stl
- link robot_base_plate: geometry collision box size=0.35 0.2 0.01; visual mesh filename=package://pa_ctrl/rviz/meshes/visual/base_plate.stl

Commit message: pipeline image traj

File: pa_ctrl/pa_ctrl/urdf/workcell.urdf (robot description, URDF)
Before this commit: robot fanuc_crx10ial, 16 links, 15 joints
Links:
- removed link camera_frame
- added link camera_R435i_link; collision mesh filename=package://pa_ctrl/rviz/meshes/collision/D435_Solid_collisio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; visual mesh filename=package://pa_ctrl/rviz/meshes/visual/D435_Solid_simple.dae
- link festool_kit: geometry collision mesh filename=package://pa_ctrl/rviz/meshes/collision/Festool_colision.dae; visual mesh filename=package://pa_ctrl/rviz/meshes/visual/Festool_v4.dae
- link husky: geometry collision mesh filename=package://pa_ctrl/rviz/meshes/collision/collision_mesh.dae; visual mesh filename=package://pa_ctrl/rviz/meshes/visual/base_mobile.dae
- link robot_base_plate: geometry collision box size=0.35 0.2 0.01; visual mesh filename=package://pa_ctrl/rviz/meshes/visual/base_plate.dae
Joints:
- removed joint world_to_camera
- added joint tool0_to_camera: type fixed, parent tool0, child camera_R435i_link, origin xyz=0.07071 -0.07071 -0.0125 rpy=1.5708 0 0.7854 
- joint tool0_to_festool_kit: origin xyz=0 0 0 rpy=0 0 0 -> xyz=0 0 0.01 rpy=0 0 2.3562

File: pa_ctrl/pa_ctrl/urdf/workcell.xacro (robot description, xacro)
@@ -56,8 +56,22 @@
   </link>
   <link name="world"/>
-  <link name="camera_frame"/>
+  <link name="camera_R435i_link">
+    <visual>
+      <origin xyz="0 0 0.0042" rpy="0 0 3.1416"/>
+      <geometry>
+        <mesh filename="package://pa_ctrl/rviz/meshes/visual/D435_Solid_simple.dae"/>
+        <!--mesh filename="package://pa_ctrl/rviz/meshes/collision/collision_mesh.dae"/-->
+      </geometry>
+    </visual>
+    <collision>
+      <origin xyz="0 0 0.0042" rpy="0 0 3.1416"/>
+      <geometry>
+        <mesh filename="package://pa_ctrl/rviz/meshes/collision/D435_Solid_collision.dae"/>
+      </geometry>
+    </collision>
+  </link>
   <!-- Diefine joint between link-->
   <joint name="tool0_to_festool_kit" type="fixed">
-    <origin xyz="0 0 0" rpy="0 0 0"/>
+    <origin xyz="0 0 0.01" rpy="0 0 2.3562"/>
     <parent link="tool0"/>
     <child  link="festool_kit"/>
@@ -86,8 +100,9 @@
     <child  link="husky"/>
   </joint>
-  <joint name="world_to_camera" type="fixed">
-    <parent link="world"/>
-    <child link="camera_frame"/>
-    <origin xyz="-0.25 -0.5 1.25" rpy="0 3.14159 0"/>
+  <joint name="tool0_to_camera" type="fixed">
+    <parent link="tool0"/>
+    <child link="camera_R435i_link"/>
+    <!-- <origin xyz="0.100 0 -0.0125" rpy="1.5708 0 1.5708 "/> -->
+    <origin xyz="0.07071 -0.07071 -0.0125" rpy="1.5708 0 0.7854 "/>
   </joint>
 </robot>

File: pa_ctrl/workcell_moveit_config/config/gazebo_fanuc_crx10ial.urdf (robot description, URDF)
Before this commit: robot fanuc_crx10ial, 16 links, 15 joints
Links:
- link festool_kit: geometry collision mesh filename=package://pa_ctrl/rviz/meshes/collision/Festool_colision.dae
- link husky: geometry 
- link robot_base_plate: geometry collision box size=0.35 0.2 0.01
Joints:
- joint joint_2: limit lower=-3.141592653589793 upper=3.141592653589793 effort=0 velocity=2.0943951023931953 -> lower=-3.141592653589793 upper=3.141592653589793 effort=100 velocity=2.0943951023931953
